File: Proyecto_Reinaldo.sch (EAGLE design)
At the start: 43 parts, among them IC2 MC34063A

Commit message: Terminado posicionado componentes BRD
Parts:
- C3: value 0.1uF -> 22pF
- C4: value 22uf -> 0.1uF; device adafruit:CPOL-USE2,5-6E -> rcl:C-USC0805
- C5: value 47uf -> 1uF; device adafruit:CPOL-USE2,5-6E -> rcl:C-USC0805
- C6: value 22pF -> 22uf; device rcl:C-USC0805 -> adafruit:CPOL-USE2,5-6E
- C8: value 1uF -> 47uf; device rcl:C-USC0805 -> adafruit:CPOL-USE2,5-6E
- R1, R10, R11, R6, R8: device rcl:R-US_R1206 -> Circuitos-Creativos-RCL:RESISTORR1206
- R12, R13, R14, R7, R9: value (none) -> 470R; device adafruit:R-US_0207/7 -> Circuitos-Creativos-RCL:RESISTORR1206
- R2, R3, R4, R5: device resistor:R-US_R1206 -> Circuitos-Creativos-RCL:RESISTORR1206
- U1: value (none) -> ATMEGA328P-AU
- renumbered U$2 to UART
Connections:
- net D5/2 renamed D5
- net D6/1 renamed D6
- net D7/4 renamed D7
- net D8/3 renamed D8
- net N$7 renamed OK3
- removed net N$3: OK2.EMIT, R8.1, X1-2.KL
- removed net N$6: OK1.EMIT, R10.1, X1-3.KL
- removed net RX1: U1.PD0(RXD), UART.1
- removed net TX0: U1.PD1(TXD), UART.3
- new net OK1: OK1.EMIT, R8.1, X1-3.KL
- new net OK2: OK2.EMIT, R10.1, X1-2.KL
- new net RX0: U1.PD0(RXD), UART.3
- new net TX1: U1.PD1(TXD), UART.1
- net +24V: now also C6.+; no longer C4.+
- net AREF: now also C4.1, U1.AREF; no longer C1.1
- net GND: now also C4.2, C5.2, C6.-, C8.-, J3.1, U1.GND; no longer C4.-, C5.-, C6.2, C8.2, J3.2
- net N$18: now also C5.1; no longer C8.1
- net OS2: now also C3.1; no longer C6.1
- net RST: now also J3.2; no longer J3.1
- net VCC: now also C1.1, C8.+; no longer C3.1, C5.+
Other:
- note added: "CON MODULO RFID"
- note removed: "conector RFID"
- moved on the sheet: C1, C3, D1, D2, IC2, ISP, J1, L3, LED1, R10, R13, R14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
